File: Breakout_DPDT/Breakout_DPDT.kicad_pcb (KiCad board)
At the start: 2 copper layers, 96 x 86 mm, 129 parts, among them J1 Conn_01x03, J2 Conn_01x03, SW1 SW_DPDT_x2

Commit message: Updated Breakout Images
Other:
- board text added: "Breadboard Compatible"
- board text added: "DPDT Push Button Breakout Boards"
Changed lines of the file:
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@@
     (effects (font (size 1 1) (thickness 0.15)))
+  )
+  (gr_text "DPDT Push Button Breakout Boards" (at 111.506 30.48) (layer "User.2")
+    (effects (font (size 3 3) (thickness 0.15)))
+  )
+  (gr_text "Breadboard Compatible" (at 111.506 36.068) (layer "User.2")
+    (effects (font (size 2 2) (thickness 0.15)))
+  )
+  (dimension (type aligned) (layer "User.2")
+    (pts (xy 160 43) (xy 160 63))
+    (height -3.83)
+    (gr_text "20.0000 mm" (at 162.68 53 90) (layer "User.2")
+      (effects (font (size 1 1) (thickness 0.15)))
+    )
+    (format (units 3) (units_format 1) (precision 4))
+    (style (thickness 0.15) (arrow_length 1.27) (text_position_mode 0) (extension_height 0.58642) (extension_offset 0.5) keep_text_aligned)
+  )
+  (dimension (type aligned) (layer "User.2")
+    (pts (xy 160 43) (xy 148 43))
+    (height 2.36)
+    (gr_text "12.0000 mm" (at 154 39.49) (layer "User.2")
+      (effects (font (size 1 1) (thickness 0.15)))
+    )
+    (format (units 3) (units_format 1) (precision 4))
+    (style (thickness 0.15) (arrow_length 1.27) (text_position_mode 0) (extension_height 0.58642) (extension_offset 0.5) keep_text_aligned)
+  )
+  (dimension (type aligned) (layer "User.2")
+    (pts (xy 64 43) (xy 64 129))
+    (height 3.548)
+    (gr_text "86.0000 mm" (at 59.302 86 90) (layer "User.2")
+      (effects (font (size 1 1) (thickness 0.15)))
+    )
+    (format (units 3) (units_format 1) (precision 4))
+    (style (thickness 0.15) (arrow_length 1.27) (text_position_mode 0) (extension_height 0.58642) (extension_offset 0.5) keep_text_aligned)
   )
   (segment (start 95.46 46.728) (end 93.428 48.76) (width 1) (layer "F.Cu") (net 1))
